Commit message: Archivos del robot Scara|
Paquetes description y bringup para revisar el control.

File: examen_description/urdf/scara_basic_position_controller.xacro (robot description, xacro)
@@ -2,5 +2,5 @@
 <robot name="robot_scara" xmlns:xacro="http://ros.org/wiki/xacro" >
     <gazebo>
-        <plugin name="joint-state_publisher_controller" filename="libgazebo_ros_joint_state_publisher.so">
+        <plugin name="joint_state_publisher_controller" filename="libgazebo_ros_joint_state_publisher.so">
             <!--update rate Hz-->
             <update_rate>10</update_rate>

File: examen_description/urdf/scara_urdf.xacro (robot description, xacro)
@@ -7,5 +7,5 @@
         <parent link="world"/>
         <child link="base_link"/>
-        <origin xyz="1 0 0" rpy="0 0 0"/>
+        <origin xyz="0 0 0" rpy="0 0 0"/>
     </joint>
     <link name="base_link">
